Commit message: fixed urdf file

File: ikSharp.Test/UR5.urdf (robot description, URDF)
Before this commit: robot UR5, 8 links, 7 joints
Joints:
- joint ee_fixed_joint: origin xyz=0.0 0.1 0.0 rpy=0.0 0.0 1.57 -> xyz=0.0 0.0823 0.0 rpy=0.0 0.0 1.57
- joint elbow_joint: axis 0.0 -1.0 0.0 -> 0.0 1.0 0.0; limit lower=-3.14 upper=3.14 effort=10.0 velocity=1.0 -> lower=-3.14 upper=3.14 effort=150.0 velocity=3.15; origin xyz=0.0 -0.1 0.5 rpy=0.0 0.0 0.0 -> xyz=0.0 -0.1197 0.42500 rpy=0.0 0.0 0.0
- joint shoulder_lift_joint: origin xyz=0.0 0.1 0.0 rpy=0.0 0.0 0.0 -> xyz=0.0 1.57075 0.0 rpy=0.0 0.13585 0.0
- joint shoulder_pan_joint: origin xyz=0.0 0.0 0.1 rpy=0.0 0.0 0.0 -> xyz=0.0 0.0 0.089159 rpy=0.0 0.0 0.0
- joint wrist_1_joint: limit lower=-3.14 upper=3.14 effort=10.0 velocity=1.0 -> lower=-6.28 upper=6.28 effort=28.0 velocity=3.2; origin xyz=0.0 0.0 0.5 rpy=0.0 0.0 0.0 -> xyz=0.0 0.0 0.39225 rpy=0.0 1.57075 0.0
- joint wrist_2_joint: limit lower=-3.14 upper=3.14 effort=10.0 velocity=1.0 -> lower=-6.28 upper=6.28 effort=28.0 velocity=3.2; origin xyz=0.0 0.1 0.0 rpy=0.0 0.0 0.0 -> xyz=0.0 0.1 0.0 rpy=0.0 0.093 0.0
- joint wrist_3_joint: limit lower=-3.14 upper=3.14 effort=10.0 velocity=1.0 -> lower=-6.28 upper=6.28 effort=28.0 velocity=3.2; origin xyz=0.0 0.0 0.1 rpy=0.0 0.0 0.0 -> xyz=0.0 0.0 0.09465 rpy=0.0 0.0 0.0

File: ikSharp.Test/UR5.urdf.xacro (robot description, xacro)
@@ -1,4 +1,4 @@
 ﻿<?xml version="1.0"?>
-<robot name="UR5" xmlns:xacro="http://ros.org/wiki/xacro">
+<robot xmlns:xacro="http://ros.org/wiki/xacro">
   <xacro:include filename="$(find ur_description)/urdf/ur.transmission.xacro" />
   <xacro:include filename="$(find ur_description)/urdf/ur.gazebo.xacro" />
